Commit message: 高保真外观：程序化曲面网格生成
把 27 台机器人的视觉外观从'基本体堆叠'升级为'程序化曲面网格'，
对应用户反馈'外观不够精细'。

主要新增
--------
- python/orolp/render/primitives.py
  曲面原语：放样 lofter、圆角箱体 rounded_box、回转体 revolve、
  锥形柱 tapered_cylinder、胶囊 capsule、扫掠管 tube
  加权面积法平滑法向 + 角度阈值 50° 保边

- python/orolp/robot_library/hifi.py
  9 个连杆的高保真配方（base / turret / upper_arm / forearm / elbow /
  wrist_roll / wrist_pitch / flange / tcp），与基本体配方签名一致
  关键改进：变截面放样主梁（肩粗肘细）、铸造圆角、J2 配重、
  侧向加强脊、背部线缆、ISO 9409 法兰定位销

接线开关
--------
- urdf_builder.py
  新增 _MeshSpec / build_mesh / _Part.mesh / _add_parts(mesh_dir)
  新增 _parts_for 在基本体与高保真间切换，_LEGACY_BUILDERS 完整保留
  build_urdf_string(spec, mesh_dir=None) 给出 mesh_dir 即写 STL

- tools/generate_robot_models.py
  --primitive 只生成零依赖 URDF；默认走 hifi 写 mesh/
  报告每台机器人的三角面数与 STL 体积

结果
----
- 28/28 通过外观校验（覆盖率 5.6%~14.0%，品牌色调匹配）
- 工业 6 轴 7144 三角面 ≈ 352 KB / 台
- 协作 6 轴 3912 三角面 ≈ 193 KB / 台
- 7 轴 iiwa  4296 三角面 ≈ 212 KB / 台
- 全套 27 台新增 7.4 MB STL，已 commit
- 38 个单元测试全部通过
- 碰撞包络仍为单基本体，SAT 代价与外观精细度解耦

File: models/abb/irb1200/irb1200.urdf (robot description, URDF)
Before this commit: robot abb_irb1200, 8 links, 7 joints
Links:
- link base_link: geometry collision cylinder length=0.108 radius=0.116046; visual mesh filename=meshes/base_link_00.stl
- link link_1: geometry collision cylinder length=0.132 radius=0.089842; visual mesh filename=meshes/link_1_00.stl
- link link_2: geometry collision box size=0.074868 0.061392 0.552; visual mesh filename=meshes/link_2_00.stl
- link link_3: geometry collision box size=0.070376 0.057708 0.432; visual mesh filename=meshes/link_3_00.stl
- link link_4: geometry collision cylinder length=0.072 radius=0.032942; visual mesh filename=meshes/link_4_00.stl
- link link_5: geometry collision box size=0.063638 0.052183 0.072; visual mesh filename=meshes/link_5_00.stl
- link tool0: geometry collision cylinder length=0.072 radius=0.031445; visual mesh filename=meshes/tool0_00.stl

File: models/abb/irb1600/irb1600.urdf (robot description, URDF)
Before this commit: robot abb_irb1600, 8 links, 7 joints
Links:
- link base_link: geometry collision cylinder length=0.108 radius=0.114115; visual mesh filename=meshes/base_link_00.stl
- link link_1: geometry collision cylinder length=0.132 radius=0.088347; visual mesh filename=meshes/link_1_00.stl
- link link_2: geometry collision box size=0.073623 0.060371 0.552; visual mesh filename=meshes/link_2_00.stl
- link link_3: geometry collision box size=0.069205 0.056748 0.432; visual mesh filename=meshes/link_3_00.stl
- link link_4: geometry collision cylinder length=0.072 radius=0.032394; visual mesh filename=meshes/link_4_00.stl
- link link_5: geometry collision box size=0.062579 0.051315 0.072; visual mesh filename=meshes/link_5_00.stl
- link tool0: geometry collision cylinder length=0.072 radius=0.030921; visual mesh filename=meshes/tool0_00.stl

File: models/abb/irb4600_20_250/irb4600_20_250.urdf (robot description, URDF)
Before this commit: robot abb_irb4600_20_250, 8 links, 7 joints
Links:
- link base_link: geometry collision cylinder length=0.2295 radius=0.132196; visual mesh filename=meshes/base_link_00.stl
- link link_1: geometry collision cylinder length=0.2805 radius=0.102345; visual mesh filename=meshes/link_1_00.stl
- link link_2: geometry collision box size=0.085287 0.069936 1.173; visual mesh filename=meshes/link_2_00.stl
- link link_3: geometry collision box size=0.08017 0.06574 0.918; visual mesh filename=meshes/link_3_00.stl
- link link_4: geometry collision cylinder length=0.153 radius=0.037526; visual mesh filename=meshes/link_4_00.stl
- link link_5: geometry collision box size=0.072494 0.059445 0.153; visual mesh filename=meshes/link_5_00.stl
- link tool0: geometry collision cylinder length=0.153 radius=0.035821; visual mesh filename=meshes/tool0_00.stl

File: models/abb/irb6700_150_320/irb6700_150_320.urdf (robot description, URDF)
Before this commit: robot abb_irb6700_150_320, 8 links, 7 joints
Links:
- link base_link: geometry collision cylinder length=0.288 radius=0.184563; visual mesh filename=meshes/base_link_00.stl
- link link_1: geometry collision cylinder length=0.352 radius=0.142887; visual mesh filename=meshes/link_1_00.stl
- link link_2: geometry collision box size=0.119073 0.09764 1.472; visual mesh filename=meshes/link_2_00.stl
- link link_3: geometry collision box size=0.111928 0.091781 1.152; visual mesh filename=meshes/link_3_00.stl
- link link_4: geometry collision cylinder length=0.192 radius=0.052392; visual mesh filename=meshes/link_4_00.stl
- link link_5: geometry collision box size=0.101212 0.082994 0.192; visual mesh filename=meshes/link_5_00.stl
- link tool0: geometry collision cylinder length=0.192 radius=0.050011; visual mesh filename=meshes/tool0_00.stl

File: models/estun/er20_1780/er20_1780.urdf (robot description, URDF)
Before this commit: robot estun_er20_1780, 8 links, 7 joints
Links:
- link base_link: geometry collision cylinder length=0.1602 radius=0.132196; visual mesh filename=meshes/base_link_00.stl
- link link_1: geometry collision cylinder length=0.1958 radius=0.102345; visual mesh filename=meshes/link_1_00.stl
- link link_2: geometry collision box size=0.085287 0.069936 0.8188; visual mesh filename=meshes/link_2_00.stl
- link link_3: geometry collision box size=0.08017 0.06574 0.6408; visual mesh filename=meshes/link_3_00.stl
- link link_4: geometry collision cylinder length=0.1068 radius=0.037526; visual mesh filename=meshes/link_4_00.stl
- link link_5: geometry collision box size=0.072494 0.059445 0.1068; visual mesh filename=meshes/link_5_00.stl
- link tool0: geometry collision cylinder length=0.1068 radius=0.035821; visual mesh filename=meshes/tool0_00.stl

File: models/estun/er50_2100/er50_2100.urdf (robot description, URDF)
Before this commit: robot estun_er50_2100, 8 links, 7 joints
Links:
- link base_link: geometry collision cylinder length=0.189 radius=0.151733; visual mesh filename=meshes/base_link_00.stl
- link link_1: geometry collision cylinder length=0.231 radius=0.117471; visual mesh filename=meshes/link_1_00.stl
- link link_2: geometry collision box size=0.097892 0.080272 0.966; visual mesh filename=meshes/link_2_00.stl
- link link_3: geometry collision box size=0.092019 0.075455 0.756; visual mesh filename=meshes/link_3_00.stl
- link link_4: geometry collision cylinder length=0.126 radius=0.043073; visual mesh filename=meshes/link_4_00.stl
- link link_5: geometry collision box size=0.083209 0.068231 0.126; visual mesh filename=meshes/link_5_00.stl
- link tool0: geometry collision cylinder length=0.126 radius=0.041115; visual mesh filename=meshes/tool0_00.stl

File: models/estun/er6_1450/er6_1450.urdf (robot description, URDF)
Before this commit: robot estun_er6_1450, 8 links, 7 joints
Links:
- link base_link: geometry collision cylinder length=0.1305 radius=0.114115; visual mesh filename=meshes/base_link_00.stl
- link link_1: geometry collision cylinder length=0.1595 radius=0.088347; visual mesh filename=meshes/link_1_00.stl
- link link_2: geometry collision box size=0.073623 0.060371 0.667; visual mesh filename=meshes/link_2_00.stl
- link link_3: geometry collision box size=0.069205 0.056748 0.522; visual mesh filename=meshes/link_3_00.stl
- link link_4: geometry collision cylinder length=0.087 radius=0.032394; visual mesh filename=meshes/link_4_00.stl
- link link_5: geometry collision box size=0.062579 0.051315 0.087; visual mesh filename=meshes/link_5_00.stl
- link tool0: geometry collision cylinder length=0.087 radius=0.030921; visual mesh filename=meshes/tool0_00.stl

File: models/fanuc/m20ia_35m/m20ia_35m.urdf (robot description, URDF)
Before this commit: robot fanuc_m20ia_35m, 8 links, 7 joints
Links:
- link base_link: geometry collision cylinder length=0.16317 radius=0.143412; visual mesh filename=meshes/base_link_00.stl
- link link_1: geometry collision cylinder length=0.19943 radius=0.111029; visual mesh filename=meshes/link_1_00.stl
- link link_2: geometry collision box size=0.092524 0.07587 0.83398; visual mesh filename=meshes/link_2_00.stl
- link link_3: geometry collision box size=0.086972 0.071317 0.65268; visual mesh filename=meshes/link_3_00.stl
- link link_4: geometry collision cylinder length=0.10878 radius=0.04071; visual mesh filename=meshes/link_4_00.stl
- link link_5: geometry collision box size=0.078645 0.064489 0.10878; visual mesh filename=meshes/link_5_00.stl
- link tool0: geometry collision cylinder length=0.10878 radius=0.03886; visual mesh filename=meshes/tool0_00.stl

File: models/fanuc/m710ic_50/m710ic_50.urdf (robot description, URDF)
Before this commit: robot fanuc_m710ic_50, 8 links, 7 joints
Links:
- link base_link: geometry collision cylinder length=0.1845 radius=0.151733; visual mesh filename=meshes/base_link_00.stl
- link link_1: geometry collision cylinder length=0.2255 radius=0.117471; visual mesh filename=meshes/link_1_00.stl
- link link_2: geometry collision box size=0.097892 0.080272 0.943; visual mesh filename=meshes/link_2_00.stl
- link link_3: geometry collision box size=0.092019 0.075455 0.738; visual mesh filename=meshes/link_3_00.stl
- link link_4: geometry collision cylinder length=0.123 radius=0.043073; visual mesh filename=meshes/link_4_00.stl
- link link_5: geometry collision box size=0.083209 0.068231 0.123; visual mesh filename=meshes/link_5_00.stl
- link tool0: geometry collision cylinder length=0.123 radius=0.041115; visual mesh filename=meshes/tool0_00.stl

File: models/fanuc/r2000ic_165f/r2000ic_165f.urdf (robot description, URDF)
Before this commit: robot fanuc_r2000ic_165f, 8 links, 7 joints
Links:
- link base_link: geometry collision cylinder length=0.23895 radius=0.188019; visual mesh filename=meshes/base_link_00.stl
- link link_1: geometry collision cylinder length=0.29205 radius=0.145563; visual mesh filename=meshes/link_1_00.stl
- link link_2: geometry collision box size=0.121302 0.099468 1.2213; visual mesh filename=meshes/link_2_00.stl
- link link_3: geometry collision box size=0.114024 0.0935 0.9558; visual mesh filename=meshes/link_3_00.stl
- link link_4: geometry collision cylinder length=0.1593 radius=0.053373; visual mesh filename=meshes/link_4_00.stl
- link link_5: geometry collision box size=0.103107 0.084548 0.1593; visual mesh filename=meshes/link_5_00.stl
- link tool0: geometry collision cylinder length=0.1593 radius=0.050947; visual mesh filename=meshes/tool0_00.stl

File: models/jaka/zu12/zu12.urdf (robot description, URDF)
Before this commit: robot jaka_zu12, 8 links, 7 joints
Links:
- link base_link: geometry collision cylinder length=0.11943 radius=0.108796; visual mesh filename=meshes/base_link_00.stl
- link link_1: geometry collision cylinder length=0.14597 radius=0.084229; visual mesh filename=meshes/link_1_00.stl
- link link_2: geometry collision box size=0.070191 0.057557 0.61042; visual mesh filename=meshes/link_2_00.stl
- link link_3: geometry collision box size=0.06598 0.054103 0.47772; visual mesh filename=meshes/link_3_00.stl
- link link_4: geometry collision cylinder length=0.07962 radius=0.030884; visual mesh filename=meshes/link_4_00.stl
- link link_5: geometry collision box size=0.059662 0.048923 0.07962; visual mesh filename=meshes/link_5_00.stl
- link tool0: geometry collision cylinder length=0.07962 radius=0.02948; visual mesh filename=meshes/tool0_00.stl

File: models/jaka/zu18/zu18.urdf (robot description, URDF)
Before this commit: robot jaka_zu18, 8 links, 7 joints
Links:
- link base_link: geometry collision cylinder length=0.09657 radius=0.114671; visual mesh filename=meshes/base_link_00.stl
- link link_1: geometry collision cylinder length=0.11803 radius=0.088778; visual mesh filename=meshes/link_1_00.stl
- link link_2: geometry collision box size=0.073981 0.060665 0.49358; visual mesh filename=meshes/link_2_00.stl
- link link_3: geometry collision box size=0.069542 0.057025 0.38628; visual mesh filename=meshes/link_3_00.stl
- link link_4: geometry collision cylinder length=0.06438 radius=0.032552; visual mesh filename=meshes/link_4_00.stl
- link link_5: geometry collision box size=0.062884 0.051565 0.06438; visual mesh filename=meshes/link_5_00.stl
- link tool0: geometry collision cylinder length=0.06438 radius=0.031072; visual mesh filename=meshes/tool0_00.stl

File: models/jaka/zu20/zu20.urdf (robot description, URDF)
Before this commit: robot jaka_zu20, 8 links, 7 joints
Links:
- link base_link: geometry collision cylinder length=0.1602 radius=0.116332; visual mesh filename=meshes/base_link_00.stl
- link link_1: geometry collision cylinder length=0.1958 radius=0.090064; visual mesh filename=meshes/link_1_00.stl
- link link_2: geometry collision box size=0.075053 0.061543 0.8188; visual mesh filename=meshes/link_2_00.stl
- link link_3: geometry collision box size=0.07055 0.057851 0.6408; visual mesh filename=meshes/link_3_00.stl
- link link_4: geometry collision cylinder length=0.1068 radius=0.033023; visual mesh filename=meshes/link_4_00.stl
- link link_5: geometry collision box size=0.063795 0.052312 0.1068; visual mesh filename=meshes/link_5_00.stl
- link tool0: geometry collision cylinder length=0.1068 radius=0.031522; visual mesh filename=meshes/tool0_00.stl

File: models/jaka/zu3/zu3.urdf (robot description, URDF)
Before this commit: robot jaka_zu3, 8 links, 7 joints
Links:
- link base_link: geometry collision cylinder length=0.05634 radius=0.093774; visual mesh filename=meshes/base_link_00.stl
- link link_1: geometry collision cylinder length=0.06886 radius=0.072599; visual mesh filename=meshes/link_1_00.stl
- link link_2: geometry collision box size=0.060499 0.049609 0.28796; visual mesh filename=meshes/link_2_00.stl
- link link_3: geometry collision box size=0.056869 0.046633 0.22536; visual mesh filename=meshes/link_3_00.stl
- link link_4: geometry collision cylinder length=0.03756 radius=0.02662; visual mesh filename=meshes/link_4_00.stl
- link link_5: geometry collision box size=0.051424 0.042168 0.03756; visual mesh filename=meshes/link_5_00.stl
- link tool0: geometry collision cylinder length=0.03756 radius=0.02541; visual mesh filename=meshes/tool0_00.stl

File: models/jaka/zu30/zu30.urdf (robot description, URDF)
Before this commit: robot jaka_zu30, 8 links, 7 joints
Links:
- link base_link: geometry collision cylinder length=0.1215 radius=0.123297; visual mesh filename=meshes/base_link_00.stl
- link link_1: geometry collision cylinder length=0.1485 radius=0.095456; visual mesh filename=meshes/link_1_00.stl
- link link_2: geometry collision box size=0.079547 0.065228 0.621; visual mesh filename=meshes/link_2_00.stl
- link link_3: geometry collision box size=0.074774 0.061315 0.486; visual mesh filename=meshes/link_3_00.stl
- link link_4: geometry collision cylinder length=0.081 radius=0.035001; visual mesh filename=meshes/link_4_00.stl
- link link_5: geometry collision box size=0.067615 0.055444 0.081; visual mesh filename=meshes/link_5_00.stl
- link tool0: geometry collision cylinder length=0.081 radius=0.03341; visual mesh filename=meshes/tool0_00.stl

File: models/jaka/zu5/zu5.urdf (robot description, URDF)
Before this commit: robot jaka_zu5, 8 links, 7 joints
Links:
- link base_link: geometry collision cylinder length=0.08586 radius=0.098521; visual mesh filename=meshes/base_link_00.stl
- link link_1: geometry collision cylinder length=0.10494 radius=0.076275; visual mesh filename=meshes/link_1_00.stl
- link link_2: geometry collision box size=0.063562 0.052121 0.43884; visual mesh filename=meshes/link_2_00.stl
- link link_3: geometry collision box size=0.059748 0.048994 0.34344; visual mesh filename=meshes/link_3_00.stl
- link link_4: geometry collision cylinder length=0.05724 radius=0.027967; visual mesh filename=meshes/link_4_00.stl
- link link_5: geometry collision box size=0.054028 0.044303 0.05724; visual mesh filename=meshes/link_5_00.stl
- link tool0: geometry collision cylinder length=0.05724 radius=0.026696; visual mesh filename=meshes/tool0_00.stl

File: models/jaka/zu7/zu7.urdf (robot description, URDF)
Before this commit: robot jaka_zu7, 8 links, 7 joints
Links:
- link base_link: geometry collision cylinder length=0.07371 radius=0.10212; visual mesh filename=meshes/base_link_00.stl
- link link_1: geometry collision cylinder length=0.09009 radius=0.079061; visual mesh filename=meshes/link_1_00.stl
- link link_2: geometry collision box size=0.065884 0.054025 0.37674; visual mesh filename=meshes/link_2_00.stl
- link link_3: geometry collision box size=0.061931 0.050783 0.29484; visual mesh filename=meshes/link_3_00.stl
- link link_4: geometry collision cylinder length=0.04914 radius=0.028989; visual mesh filename=meshes/link_4_00.stl
- link link_5: geometry collision box size=0.056001 0.045921 0.04914; visual mesh filename=meshes/link_5_00.stl
- link tool0: geometry collision cylinder length=0.04914 radius=0.027671; visual mesh filename=meshes/tool0_00.stl

File: models/kuka/kr16_2/kr16_2.urdf (robot description, URDF)
Before this commit: robot kuka_kr16_2, 8 links, 7 joints
Links:
- link base_link: geometry collision cylinder length=0.14499 radius=0.128275; visual mesh filename=meshes/base_link_00.stl
- link link_1: geometry collision cylinder length=0.17721 radius=0.09931; visual mesh filename=meshes/link_1_00.stl
- link link_2: geometry collision box size=0.082758 0.067862 0.74106; visual mesh filename=meshes/link_2_00.stl
- link link_3: geometry collision box size=0.077792 0.06379 0.57996; visual mesh filename=meshes/link_3_00.stl
- link link_4: geometry collision cylinder length=0.09666 radius=0.036413; visual mesh filename=meshes/link_4_00.stl
- link link_5: geometry collision box size=0.070344 0.057682 0.09666; visual mesh filename=meshes/link_5_00.stl
- link tool0: geometry collision cylinder length=0.09666 radius=0.034758; visual mesh filename=meshes/tool0_00.stl

File: models/kuka/kr20_r1810/kr20_r1810.urdf (robot description, URDF)
Before this commit: robot kuka_kr20_r1810, 8 links, 7 joints
Links:
- link base_link: geometry collision cylinder length=0.16317 radius=0.132196; visual mesh filename=meshes/base_link_00.stl
- link link_1: geometry collision cylinder length=0.19943 radius=0.102345; visual mesh filename=meshes/link_1_00.stl
- link link_2: geometry collision box size=0.085287 0.069936 0.83398; visual mesh filename=meshes/link_2_00.stl
- link link_3: geometry collision box size=0.08017 0.06574 0.65268; visual mesh filename=meshes/link_3_00.stl
- link link_4: geometry collision cylinder length=0.10878 radius=0.037526; visual mesh filename=meshes/link_4_00.stl
- link link_5: geometry collision box size=0.072494 0.059445 0.10878; visual mesh filename=meshes/link_5_00.stl
- link tool0: geometry collision cylinder length=0.10878 radius=0.035821; visual mesh filename=meshes/tool0_00.stl

File: models/kuka/kr210_r2700/kr210_r2700.urdf (robot description, URDF)
Before this commit: robot kuka_kr210_r2700, 8 links, 7 joints
Links:
- link base_link: geometry collision cylinder length=0.24309 radius=0.19727; visual mesh filename=meshes/base_link_00.stl
- link link_1: geometry collision cylinder length=0.29711 radius=0.152725; visual mesh filename=meshes/link_1_00.stl
- link link_2: geometry collision box size=0.127271 0.104362 1.24246; visual mesh filename=meshes/link_2_00.stl
- link link_3: geometry collision box size=0.119635 0.0981 0.97236; visual mesh filename=meshes/link_3_00.stl
- link link_4: geometry collision cylinder length=0.16206 radius=0.055999; visual mesh filename=meshes/link_4_00.stl
- link link_5: geometry collision box size=0.10818 0.088708 0.16206; visual mesh filename=meshes/link_5_00.stl
- link tool0: geometry collision cylinder length=0.16206 radius=0.053454; visual mesh filename=meshes/tool0_00.stl
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